File: programmer-smd.brd (EAGLE design)
At the start: 17.8 x 30.5 mm, 10 parts, among them IC1 TINY13-20PU

Commit message: Added copyright
Parts:
- R1: value 1k -> 100
Other:
- outline, holes or cut-outs redrawn
- board text added: "(C) 2016 Sarif Software"
- board text added: "IC"
- board text added: "programmer"
- board text added: "rev A"
Changed lines of the file:
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@@
 <board>
 <plain>
-<wire x1="0" y1="0" x2="17.7675" y2="0" width="0" layer="20"/>
-<wire x1="17.7675" y1="0" x2="17.7675" y2="30.47" width="0" layer="20"/>
-<wire x1="17.7675" y1="30.47" x2="0" y2="30.47" width="0" layer="20"/>
-<wire x1="0" y1="30.47" x2="0" y2="0" width="0" layer="20"/>
 <text x="2.54" y="5.715" size="0.8128" layer="23" font="vector" rot="R90" align="center-left">GND</text>
 <text x="5.08" y="5.715" size="0.8128" layer="23" font="vector" rot="R90" align="center-left">SCLK</text>
@@
 <text x="10.16" y="28.575" size="0.8128" layer="23" font="vector" rot="R90" align="center-left">6</text>
 <text x="12.7" y="28.575" size="0.8128" layer="23" font="vector" rot="R90" align="center-left">5</text>
-<circle x="2.54" y="17.145" radius="0.635" width="0.254" layer="23"/>
+<circle x="2.54" y="16.51" radius="0.635" width="0.254" layer="23"/>
+<wire x1="0" y1="26.035" x2="0" y2="1.905" width="0" layer="20"/>
+<wire x1="4.445" y1="30.48" x2="0" y2="26.035" width="0" layer="20"/>
+<wire x1="13.335" y1="30.48" x2="17.78" y2="26.035" width="0" layer="20"/>
+<wire x1="17.78" y1="26.035" x2="17.78" y2="1.905" width="0" layer="20"/>
+<wire x1="4.445" y1="30.48" x2="13.335" y2="30.48" width="0" layer="20"/>
+<text x="8.89" y="19.05" size="1.778" layer="23" font="vector" align="center">IC</text>
+<wire x1="0" y1="1.905" x2="1.905" y2="0" width="0" layer="20"/>
+<wire x1="1.905" y1="0" x2="15.875" y2="0" width="0" layer="20"/>
+<wire x1="17.78" y1="1.905" x2="15.875" y2="0" width="0" layer="20"/>
+<text x="13.97" y="20.32" size="1.27" layer="24" font="vector" rot="MR0" align="center-left">programmer</text>
+<text x="13.97" y="19.05" size="0.6096" layer="24" font="vector" rot="MR0" align="center-left">rev A</text>
+<text x="14.605" y="17.145" size="0.6096" layer="24" font="vector" rot="MR0" align="center-left">(C) 2016 Sarif Software</text>
 </plain>
 <attributes>
@@
 <attribute name="OC_FARNELL" value="unknown" x="34.29" y="-12.7" size="1.778" layer="27" display="off"/>
 </element>
-<element name="R1" library="resistor" package="M0805" value="1k" x="15.24" y="13.335" rot="R90"/>
+<element name="R1" library="resistor" package="M0805" value="100" x="15.24" y="13.335" rot="R90"/>
 <element name="LED1" library="led" package="CHIP-LED0805" value="" x="15.24" y="19.05" rot="R180"/>
 </elements>
