File: programmer-smd.sch (EAGLE design)
At the start: 10 parts, among them IC1 TINY13-20PU

Commit message: Added copyright
Parts:
- R1: value 1k -> 100
Changed lines of the file:
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@@
 <part name="R5" library="resistor" deviceset="R-US_" device="M0805" value="1k"/>
 <part name="RASPBERRYPI_GPIO" library="parts" deviceset="MA06-1" device=""/>
-<part name="R1" library="resistor" deviceset="R-US_" device="M0805" value="1k"/>
+<part name="R1" library="resistor" deviceset="R-US_" device="M0805" value="100"/>
 <part name="LED1" library="led" deviceset="LED" device="CHIP-LED0805"/>
 </parts>
